Commit message: [update] modify b0 to world

File: urdf/zzz_arm.urdf (robot description, URDF)
Before this commit: robot zzz_arm, 4 links, 3 joints
Links:
- removed link b0
- added link world
Joints:
- joint j0: origin xyz=2.0 0 0 -> xyz=1 1 0; parent b0 -> world

Commit message: [update] add b4 as end link

File: urdf/zzz_arm.urdf (robot description, URDF)
Before this commit: robot zzz_arm, 4 links, 3 joints
Links:
- added link b4
Joints:
- added joint j3: type revolute, parent b3, child b4, origin xyz=2.0 0 0, axis 0 0 1, limit lower=-3.14 upper=3.14 effort=1.0 velocity=3.14

Commit message: [update] to set end link to be fixed

File: urdf/zzz_arm.urdf (robot description, URDF)
Before this commit: robot zzz_arm, 5 links, 4 joints
Joints:
- joint j3: axis 0 0 1 -> (none); limit lower=-3.14 upper=3.14 effort=1.0 velocity=3.14 -> (none); type revolute -> fixed

Commit message: [update] zzz arm

File: urdf/zzz_arm.urdf (robot description, URDF)
Before this commit: robot zzz_arm, 5 links, 4 joints
Joints:
- joint j0: origin xyz=1 1 0 -> xyz=2.0 0 0
